File: nesceptor/pcb/inconsole/inconsole.kicad_pcb (KiCad board)
At the start: 2 copper layers, 0 parts

Commit message: Add NES CPU on back side and initial edge cut
More space could be available to the left, but want to avoid RF
shielding if at all possible. This is because when you remove the RF
shielding and don't put it back - you're probably going to lose it and
that is essentially modifying the console.

To the right there are pins from a capacitor that should be left alone.
Parts:
- added U1: ~, argos:DIP-40_W15.24mm_Castellated, B.Cu at (82.9, 74.6)
Other:
- board outline added: 63.5 x 15.2 mm
